File: Hardware/PCB/KiCad_Files/HydrogelBioprinter/Control.kicad_sch (KiCad schematic)
At the start: 42 parts, among them J26 Screw_Terminal_01x02, J27 Screw_Terminal_01x02, J28 Screw_Terminal_01x02, J29 Screw_Terminal_01x02, Q5 RFP30N06LE, Q7 RFP30N06LE, Q8 RFP30N06LE, Q9 RFP30N06LE, U7 SN74HC245DWR

Commit message: Schematic Update, PCB preliminary layout, Machine Design addition, and LaTeX report addition
Parts:
- removed D2: SMAJ28A, Diode_SMD:D_SMA, symbol Diode:SMAJ28A
- removed R11, R14, R19, R22: 47R, symbol Device:R
- added D11: SMAJ16A, Diode_SMD:D_SMA, symbol Diode:SMAJ16A
- C47: renamed from C31; footprint (none) -> Capacitor_SMD:C_0603_1608Metric
- J41: renamed from J28; footprint (none) -> TerminalBlock_Phoenix:TerminalBlock_Phoenix_MKDS-1,5-2-5.08_1x02_P5.08mm_Horizontal
- J42: renamed from J29; footprint (none) -> TerminalBlock_Phoenix:TerminalBlock_Phoenix_MKDS-1,5-2-5.08_1x02_P5.08mm_Horizontal
- J43: renamed from J27; footprint (none) -> TerminalBlock_Phoenix:TerminalBlock_Phoenix_MKDS-1,5-2-5.08_1x02_P5.08mm_Horizontal
- J44: renamed from J26; footprint (none) -> TerminalBlock_Phoenix:TerminalBlock_Phoenix_MKDS-1,5-2-5.08_1x02_P5.08mm_Horizontal
- R23, R24: footprint (none) -> Resistor_SMD:R_0805_2012Metric
- R25: renamed from R27; footprint (none) -> Resistor_SMD:R_0805_2012Metric
- R26, R40: renamed from R12; footprint (none) -> Resistor_SMD:R_0805_2012Metric
- R27: renamed from R21; footprint (none) -> Resistor_SMD:R_0805_2012Metric
- R28: renamed from R31; footprint (none) -> Resistor_THT:R_Axial_DIN0207_L6.3mm_D2.5mm_P10.16mm_Horizontal
- R29: renamed from R20; footprint (none) -> Resistor_SMD:R_0805_2012Metric
- R30: renamed from R25; footprint (none) -> Resistor_SMD:R_0805_2012Metric
- R31: renamed from R11; footprint (none) -> Resistor_SMD:R_0805_2012Metric
- R32: renamed from R26; footprint (none) -> Resistor_SMD:R_0805_2012Metric
- R33: renamed from R28; footprint (none) -> Resistor_SMD:R_0805_2012Metric
- R34: renamed from R18; footprint (none) -> Resistor_SMD:R_0805_2012Metric
- R35: renamed from R17; footprint (none) -> Resistor_SMD:R_0805_2012Metric
- R36: renamed from R3; footprint (none) -> Resistor_SMD:R_0805_2012Metric
- R37: renamed from R4; footprint (none) -> Resistor_SMD:R_0805_2012Metric
- R38: renamed from R29; footprint (none) -> Resistor_SMD:R_0805_2012Metric
- R39: renamed from R9; footprint (none) -> Resistor_SMD:R_0805_2012Metric
- R41: renamed from R13; footprint (none) -> Resistor_SMD:R_0805_2012Metric
- R42: renamed from R16; footprint (none) -> Resistor_SMD:R_0805_2012Metric
- R43: renamed from R15; footprint (none) -> Resistor_SMD:R_0805_2012Metric
- R44: renamed from R10; footprint (none) -> Resistor_SMD:R_0805_2012Metric
- R45: renamed from R30; footprint (none) -> Resistor_SMD:R_0805_2012Metric
- renumbered C32 to C18, C33 to C19, C34 to C48, C35 to C49, Q8 to Q3, Q9 to Q4, Q7 to Q5, Q5 to Q6
Connections:
- net +12V: now also D11.1 (A1)
- net GND: now also D11.2 (A2)
- net at R27.2, U7.8 (A7): now also U7.9 (A8)
- net at U7.6 (A5): now also R29.2, U7.7 (A6)
- net at U7.2 (A1): now also R40.2, U7.3 (A2)
- net at R41.2, U7.4 (A3): now also U7.5 (A4)
Other:
- note added: "Series Resistors that are high enough to limit the gate discharge current while still low enough to have a faster rise time"
- note added: "The HC245 is used to drive the gates of the MOSFETs so that it can act as a buffer and sink the gate discharge current instead of the STM32"
- note added: "Two buffer output channels are used to allow it to be able to sink double the amount of current"
