File: Hardware/PCB/KiCad_Files/HydrogelBioprinter/Feedback.kicad_sch (KiCad schematic)
At the start: 25 parts, among them J30 Screw_Terminal_01x02, J31 Screw_Terminal_01x02, J32 Screw_Terminal_01x02, J33 Screw_Terminal_01x02, J34 Screw_Terminal_01x02, J35 Screw_Terminal_01x02, J36 Screw_Terminal_01x02, J37 Screw_Terminal_01x02, J38 Screw_Terminal_01x05, Q10 MMBT4403_, U5 MAX6675ISA_, U6 TMUX1208PWR, U9 HX711

Commit message: Schematic Update, PCB preliminary layout, Machine Design addition, and LaTeX report addition
Parts:
- added C38: 10u, Capacitor_SMD:C_0805_2012Metric, symbol Device:C
- added C42: 100n, Capacitor_SMD:C_0603_1608Metric, symbol Device:C
- added R21, R22: 100R, Resistor_SMD:R_0603_1608Metric, symbol Device:R
- C36: renamed from C38; footprint Capacitor_SMD:C_0402_1005Metric -> Capacitor_SMD:C_0603_1608Metric
- C37: renamed from C36; footprint Capacitor_SMD:C_0402_1005Metric -> Capacitor_SMD:C_0603_1608Metric
- C39, C40: footprint Capacitor_SMD:C_0402_1005Metric -> Capacitor_SMD:C_0603_1608Metric
- C41: footprint (none) -> Capacitor_SMD:C_0805_2012Metric
- C43: renamed from C37; footprint Capacitor_SMD:C_0402_1005Metric -> Capacitor_SMD:C_0603_1608Metric
- C44: renamed from C42; footprint Capacitor_SMD:C_0402_1005Metric -> Capacitor_SMD:C_0603_1608Metric
- J32: renamed from J38; footprint (none) -> TerminalBlock_Phoenix:TerminalBlock_Phoenix_PT-1,5-5-3.5-H_1x05_P3.50mm_Horizontal
- J33: renamed from J30; footprint (none) -> TerminalBlock_Phoenix:TerminalBlock_Phoenix_PT-1,5-2-3.5-H_1x02_P3.50mm_Horizontal
- J34: renamed from J31; footprint (none) -> TerminalBlock_Phoenix:TerminalBlock_Phoenix_PT-1,5-2-3.5-H_1x02_P3.50mm_Horizontal
- J35: renamed from J32; footprint (none) -> TerminalBlock_Phoenix:TerminalBlock_Phoenix_PT-1,5-2-3.5-H_1x02_P3.50mm_Horizontal
- J36: renamed from J33; footprint (none) -> TerminalBlock_Phoenix:TerminalBlock_Phoenix_PT-1,5-2-3.5-H_1x02_P3.50mm_Horizontal
- J37: renamed from J34; footprint (none) -> TerminalBlock_Phoenix:TerminalBlock_Phoenix_PT-1,5-2-3.5-H_1x02_P3.50mm_Horizontal
- J38: renamed from J35; footprint (none) -> TerminalBlock_Phoenix:TerminalBlock_Phoenix_PT-1,5-2-3.5-H_1x02_P3.50mm_Horizontal
- J39: renamed from J36; footprint (none) -> TerminalBlock_Phoenix:TerminalBlock_Phoenix_PT-1,5-2-3.5-H_1x02_P3.50mm_Horizontal
- J40: renamed from J37; footprint (none) -> TerminalBlock_Phoenix:TerminalBlock_Phoenix_PT-1,5-2-3.5-H_1x02_P3.50mm_Horizontal
- JP6: renamed from JP2; footprint (none) -> TestPoint:TestPoint_Bridge_Pitch2.54mm_Drill0.7mm
- L2: footprint (none) -> Inductor_SMD:L_0805_2012Metric
- R18: renamed from R32; footprint (none) -> Resistor_SMD:R_0805_2012Metric
- R19: renamed from R33; footprint (none) -> Resistor_SMD:R_0805_2012Metric
- R20: renamed from R34; footprint (none) -> Resistor_SMD:R_0805_2012Metric
- renumbered Q10 to Q2, U9 to U4
Connections:
- net +3.3V: now also C38.2
- net GND: now also C38.1
- net at U4.8 (INA+): now also R21.1; no longer J32.2 (Pin_2)
- net at U4.7 (INA-): now also R22.1; no longer J32.3 (Pin_3)
- new net: C42.1, J32.3 (Pin_3), R22.2
- new net: C42.2, J32.2 (Pin_2), R21.2
Other:
- note added: "Analogue MUX to select one thermocouple at a time to be sampled by the MCU after signal conditioning"
- note added: "BLACK"
- note added: "GREEN"
- note added: "RED"
- note added: "This circuit is used to condition the load cell signal and produce a digital output for MCU sampling"
- note added: "This is used to amplify the thermocouple signal and turn it into a digital one for sampling by the STM32"
- note added: "This load cell schematic is based on the Sparkfun HX711 Load Cell breakout board"
- note added: "VBG=1.25V"
- note added: "WHITE"
- note added: "YELLOW"

Commit message: Gantry Concept 1 Completion and PCB schematic update
Changed lines of the file:
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@@
+	)
+	(junction
+		(at 233.68 104.14)
+		(diameter 0)
+		(color 0 0 0 0)
 	)
 	(junction
@@
 	(junction
 		(at 233.68 111.76)
-		(diameter 0)
-		(color 0 0 0 0)
-	)
-	(junction
-		(at 233.68 104.14)
 		(diameter 0)
 		(color 0 0 0 0)
@@
 	(wire
 		(pts
+			(xy 233.68 104.14) (xy 233.68 109.855)
+		)
+		(stroke
+			(width 0)
+			(type default)
+		)
+	)
+	(wire
+		(pts
 			(xy 40.64 111.76) (xy 49.53 111.76)
 		)
@@
 		)
 		(stroke
-			(width 0)
-			(type default)
-		)
-	)
-	(wire
-		(pts
-			(xy 233.68 109.855) (xy 233.68 104.14)
-		)
-		(stroke

Commit message: Rough PCB Design Completion
Connections:
- net GND: now also J32.2 (Pin_2), J32.5 (Pin_5); no longer J32.1 (Pin_1), J32.4 (Pin_4)
- net at C41.1, C44.1, L2.2: now also J32.1 (Pin_1); no longer J32.5 (Pin_5)
- net at C42.2, R21.2: now also J32.4 (Pin_4); no longer J32.2 (Pin_2)
Other:
- moved on the sheet: J32
Changed lines of the file:
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@@
 	(symbol
 		(lib_id "Connector:Screw_Terminal_01x05")
-		(at 228.6 120.65 270)
+		(at 228.6 120.65 90)
+		(mirror x)
 		(unit 1)
 		(exclude_from_sim no)
@@
 		(dnp no)
 		(property "Reference" "J32"
-			(at 217.932 118.618 90)
+			(at 219.075 119.38 90)
 			(effects
 				(font
@@
 		)
 		(property "Value" "Screw_Terminal_01x05"
-			(at 209.042 121.158 90)
+			(at 210.185 121.92 90)
 			(effects
 				(font

Commit message: Final PCB Design
Parts:
- JP6: footprint TestPoint:TestPoint_Bridge_Pitch2.54mm_Drill0.7mm -> TestPoint:TestPoint_2Pads_Pitch2.54mm_Drill0.8mm
Changed lines of the file:
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@@
 			)
 		)
-		(property "Footprint" "TestPoint:TestPoint_Bridge_Pitch2.54mm_Drill0.7mm"
+		(property "Footprint" "TestPoint:TestPoint_2Pads_Pitch2.54mm_Drill0.8mm"
 			(at 252.73 46.99 0)
 			(effects
