File: Hardware/PCB/KiCad_Files/HydrogelBioprinter/HydrogelBioprinter.kicad_sch (KiCad schematic)
At the start: 39 parts, among them J1 USB_B_Micro, J2 Conn_01x04_Pin, SW1 SW_Push, SW2 SW_SPDT, U1 STM32F407VGT6, U2 M24C64-WMN6TP, Y1 16MHz

Commit message: Schematic Update, PCB preliminary layout, Machine Design addition, and LaTeX report addition
Parts:
- removed C12: 1u, symbol Device:C
- removed C13: 10n, Capacitor_SMD:C_0402_1005Metric, symbol Device:C
- removed J2: Conn_01x04_Pin, symbol Connector:Conn_01x04_Pin
- added H1, H2, H3, H4: MountingHole_Pad, MountingHole:MountingHole_3.2mm_M3_Pad, symbol Mechanical:MountingHole_Pad
- added J10, J11, J12, J13, J14, J7, J8, J9: Conn, Connector_Wire:SolderWire-0.75sqmm_1x01_D1.25mm_OD3.5mm, symbol Connector_Generic:Conn_01x01
- added J16: Conn_02x05_Odd_Even, Connector_PinHeader_2.54mm:PinHeader_2x05_P2.54mm_Vertical_SMD, symbol Connector_Generic:Conn_02x05_Odd_Even
- added R14, R15: 22, Resistor_SMD:R_0603_1608Metric, symbol Device:R
- C10: renamed from C5; footprint Capacitor_SMD:C_0402_1005Metric -> Capacitor_SMD:C_0603_1608Metric
- C11: renamed from C4; footprint Capacitor_SMD:C_0402_1005Metric -> Capacitor_SMD:C_0603_1608Metric
- C12: renamed from C3; footprint Capacitor_SMD:C_0402_1005Metric -> Capacitor_SMD:C_0603_1608Metric
- C13: renamed from C2; footprint Capacitor_SMD:C_0402_1005Metric -> Capacitor_SMD:C_0603_1608Metric
- C14: renamed from C1; footprint Capacitor_SMD:C_0402_1005Metric -> Capacitor_SMD:C_0603_1608Metric
- C15: renamed from C9; footprint (none) -> Capacitor_SMD:C_0603_1608Metric
- C16: renamed from C10; footprint (none) -> Capacitor_SMD:C_0805_2012Metric
- C17: renamed from C11; footprint (none) -> Capacitor_SMD:C_0805_2012Metric
- C20: renamed from C14; footprint Capacitor_SMD:C_0402_1005Metric -> Capacitor_SMD:C_0603_1608Metric
- C21: renamed from C15; footprint (none) -> Capacitor_SMD:C_0402_1005Metric
- C22: renamed from C16; footprint (none) -> Capacitor_SMD:C_0402_1005Metric
- C23: renamed from C20; footprint Capacitor_SMD:C_0402_1005Metric -> Capacitor_SMD:C_0603_1608Metric
- C24: renamed from C17; footprint (none) -> Capacitor_SMD:C_0805_2012Metric
- C25: renamed from C18; footprint (none) -> Capacitor_SMD:C_0805_2012Metric
- C6: renamed from C19; footprint Capacitor_SMD:C_0402_1005Metric -> Capacitor_SMD:C_0603_1608Metric
- C7: renamed from C8; footprint (none) -> Capacitor_SMD:C_0805_2012Metric
- C8: renamed from C7; footprint Capacitor_SMD:C_0402_1005Metric -> Capacitor_SMD:C_0603_1608Metric
- C9: renamed from C6; footprint Capacitor_SMD:C_0402_1005Metric -> Capacitor_SMD:C_0603_1608Metric
- D5: renamed from D1; footprint (none) -> LED_SMD:LED_0805_2012Metric
- FB1: footprint (none) -> Inductor_SMD:L_0805_2012Metric
- J15: renamed from J1; footprint (none) -> Connector_USB:USB_Micro-B_Molex-105017-0001
- R10: renamed from R5; footprint (none) -> Resistor_SMD:R_0805_2012Metric
- R11: renamed from R6; footprint (none) -> Resistor_SMD:R_0805_2012Metric
- R12: renamed from R7; footprint (none) -> Resistor_SMD:R_0805_2012Metric
- R13: renamed from R8; footprint (none) -> Resistor_SMD:R_0805_2012Metric
- R16: renamed from R9; value 510R -> 470R; footprint (none) -> Resistor_THT:R_Axial_DIN0207_L6.3mm_D2.5mm_P10.16mm_Horizontal
- R6: renamed from R1; footprint (none) -> Resistor_SMD:R_0805_2012Metric
- R7: renamed from R3; footprint (none) -> Resistor_SMD:R_0805_2012Metric
- R8: renamed from R4; footprint (none) -> Resistor_SMD:R_0805_2012Metric
- R9: renamed from R2; footprint (none) -> Resistor_SMD:R_0805_2012Metric
- SW1: renamed from SW2; footprint (none) -> Button_Switch_SMD:SW_SPDT_PCM12
- SW2: renamed from SW1; footprint (none) -> Button_Switch_THT:SW_PUSH_6mm
- Y1: footprint (none) -> Crystal:Crystal_SMD_3225-4Pin_3.2x2.5mm
- renumbered U1 to U3
Connections:
- net MISO_SD is gone; now on net SPI1_MISO_SD: Card1.7 (DAT0(D0)), R12.2
- net MOSI_SD is gone; now on net SPI1_MOSI_SD: Card1.3 (CMD(DI)), R10.2
- net SCK_SD is gone; now on net SPI1_SCK_SD: Card1.5 (CLK(SCLK))
- net SCL_EEPROM is gone; now on net I2C2_SCL_EEPROM: R8.2, U2.6 (SCL)
- net SDA_EEPROM is gone; now on net I2C2_SDA_EEPROM: R7.1, U2.5 (SDA)
- net +3.3V: now also J16.1 (Pin_1)
- net A0_T: now also U3.55 (PD8)
- net A1_T: now also U3.56 (PD9)
- net A2_T: now also U3.57 (PD10)
- net CD_SD: now also U3.33 (PC4)
- net CS_SD: now also U3.29 (PA4)
- net DAT_L: now also U3.59 (PD12)
- net DIR1: now also U3.39 (PE8)
- net DIR2: now also U3.41 (PE10)
- net DIR3: now also U3.43 (PE12)
- net DIR4: now also U3.46 (PE15)
- net DIR5: now also U3.34 (PC5)
- net EN_FAN: now also U3.92 (PB6)
- net EN_Heater: now also U3.91 (PB5)
- net EN_Peltier: now also U3.90 (PB4)
- net EN_T: now also U3.54 (PB15)
- net EN_UV: now also U3.93 (PB7)
- net GND: now also H1.1, H2.1, H3.1, H4.1, J10.1 (Pin_1), J12.1 (Pin_1), J14.1 (Pin_1), J16.3 (Pin_3), J16.5 (Pin_5), J16.9 (Pin_9), J8.1 (Pin_1)
- net M0: now also U3.36 (PB1)
- net M1: now also U3.37 (PB2)
- net NRST: now also J16.10 (Pin_10)
- net SCK_L: now also U3.58 (PD11)
- net STEP1: now also U3.40 (PE9)
- net STEP2: now also U3.42 (PE11)
- net STEP3: now also U3.44 (PE13)
- net STEP4: now also U3.45 (PE14)
- net STEP5: now also U3.26 (PA3)
- net SWCLK: now also J16.4 (Pin_4)
- net SWDIO: now also R14.2
- net ~{CS_T}: now also U3.51 (PB12)
- net ~{EN}: now also U3.38 (PE7)
- net GPIO3: now reaches U3.1 (PE2)
- net at U3.15 (PC0): now also J7.1 (Pin_1)
- net at U3.16 (PC1): now also J9.1 (Pin_1)
- net at U3.17 (PC2): now also J11.1 (Pin_1)
- net at U3.18 (PC3): now also J13.1 (Pin_1)
- net GPIO4: now reaches U3.2 (PE3)
- net ADC_IN0: now reaches U3.23 (PA0)
- net ADC_IN1: now reaches U3.24 (PA1)
- net ADC_IN2: now reaches U3.25 (PA2)
- net GPIO5: now reaches U3.3 (PE4)
- net SPI1_SCK_SD: now reaches U3.30 (PA5)
- net SPI1_MISO_SD: now reaches U3.31 (PA6)
- net SPI1_MOSI_SD: now reaches U3.32 (PA7)
- net GPIO6: now reaches U3.4 (PE5)
- net I2C2_SCL_EEPROM: now reaches U3.47 (PB10)
- net I2C2_SDA_EEPROM: now reaches U3.48 (PB11)
- net GPIO7: now reaches U3.5 (PE6)
- net SPI2_SCK_T: now reaches U3.52 (PB13)
- net SPI2_MISO_T: now reaches U3.53 (PB14)
- net USART1_TX: now reaches U3.68 (PA9)
- net USART1_RX: now reaches U3.69 (PA10)
- net SPI3_CK: now reaches U3.78 (PC10)
- net SPI3_MISO: now reaches U3.79 (PC11)
- net SPI3__MOSI: now reaches U3.80 (PC12)
- net USART2_TX: now reaches U3.86 (PD5)
- net USART2_RX: now reaches U3.87 (PD6)
- net SWO: now reaches U3.89 (PB3)
- net SWO: now also R15.2
- net I2C1_SCL: now reaches U3.95 (PB8)
- net I2C1_SDA: now reaches U3.96 (PB9)
- net GPIO1: now reaches U3.97 (PE0)
- net GPIO2: now reaches U3.98 (PE1)
- net +5V: now reaches D5.2 (A), J15.1 (VBUS)
- new net: J16.6 (Pin_6), R15.1
- new net: J16.2 (Pin_2), R14.1
- no-connect marks 4 -> 25
Other:
- sheet Control Circuit ports: added EN_FAN, EN_Heater, EN_Peltier, EN_UV; removed none
- sheet Feedback Circuit ports: added A0_T, A1_T, A2_T, DAT_L, EN_T, MISO_T, SCK_L, SCK_T, ~{CS_T}; removed none
- sheet Stepper Drivers ports: added DIR1, DIR2, DIR3, DIR4, DIR5, M0, M1, STEP1, STEP2, STEP3, STEP4, STEP5, ~{EN}; removed none
- note added: "Connecters for limit switches"
- note added: "MOUNTING HOLES"
- note removed: "VREF+ Filtering"
- moved on the sheet: C10, C11, C12, C13, C14, C15, C16, C17, C20, C21, C22, C23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

Commit message: Gantry Concept 2 Completion
Connections:
- net ~{RESET}: now reaches U3.63 (PC6)
- net ~{SLEEP}: now reaches U3.64 (PC7)
- net M2: now reaches U3.65 (PC8)
- no-connect marks 25 -> 22
Other:
- sheet Stepper Drivers ports: added M2, ~{RESET}, ~{SLEEP}; removed none
Changed lines of the file:
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@@
 	)
 	(no_connect
-		(at 135.89 152.4)
-	)
-	(no_connect
 		(at 261.62 149.86)
 	)
@@
 	)
 	(no_connect
-		(at 135.89 149.86)
-	)
-	(no_connect
 		(at 231.14 91.44)
 	)
@@
 	)
 	(no_connect
-		(at 135.89 147.32)
-	)
-	(no_connect
 		(at 85.09 116.84)
 	)
@@
 	(wire
 		(pts
+			(xy 33.02 118.11) (xy 39.37 118.11)
+		)
+		(stroke
+			(width 0)
+			(type default)
+		)
+	)
+	(wire
+		(pts
 			(xy 278.13 38.1) (xy 278.13 40.64)
 		)
@@
 	(wire
 		(pts
+			(xy 33.02 110.49) (xy 39.37 110.49)
+		)
+		(stroke
+			(width 0)
+			(type default)
+		)
+	)
+	(wire
+		(pts
 			(xy 135.89 73.66) (xy 138.43 73.66)
 		)
@@
 	(wire
 		(pts
+			(xy 33.02 107.95) (xy 39.37 107.95)
+		)
+		(stroke
+			(width 0)
+			(type default)
+		)
+	)
+	(wire
+		(pts
 			(xy 60.96 68.58) (xy 67.31 68.58)
 		)
@@
 	(wire
 		(pts
+			(xy 135.89 147.32) (xy 138.43 147.32)
+		)
+		(stroke
+			(width 0)
+			(type default)
+		)
+	)
+	(wire
+		(pts
 			(xy 135.89 76.2) (xy 138.43 76.2)
 		)
@@
 	(wire
 		(pts
+			(xy 135.89 149.86) (xy 138.43 149.86)
+		)
+		(stroke
+			(width 0)
+			(type default)
+		)
+	)
+	(wire
+		(pts
 			(xy 152.4 24.13) (xy 153.67 24.13)
 		)
@@
 	(wire
 		(pts
+			(xy 135.89 152.4) (xy 138.43 152.4)
+		)
+		(stroke
+			(width 0)
+			(type default)
+		)
+	)
+	(wire
+		(pts
 			(xy 269.24 86.36) (xy 273.05 86.36)
 		)
@@
 	(wire
 		(pts
-			(xy 33.02 106.68) (xy 39.37 106.68)
+			(xy 33.02 105.41) (xy 39.37 105.41)
 		)
 		(stroke
@@
 		)
 	)
+	(global_label "M2"
+		(shape input)
+		(at 138.43 152.4 0)
+		(fields_autoplaced yes)
+		(effects
+			(font
+				(size 1.27 1.27)
+			)
+			(justify left)
+		)
+		(property "Intersheetrefs" "${INTERSHEET_REFS}"
+			(at 144.0761 152.4 0)
+			(effects
+				(font
+					(size 1.27 1.27)
+				)
+				(justify left)
+				(hide yes)
+			)
+		)
+	)
 	(global_label "STEP2"
 		(shape input)
@@
 		)
 	)
+	(global_label "~{RESET}"
+		(shape input)
+		(at 39.37 110.49 0)
+		(fields_autoplaced yes)
+		(effects
+			(font
+				(size 1.27 1.27)
+			)
+			(justify left)
+		)
+		(property "Intersheetrefs" "${INTERSHEET_REFS}"
+			(at 48.1003 110.49 0)
+			(effects
+				(font
+					(size 1.27 1.27)
+				)
+				(justify left)
+				(hide yes)
+			)
+		)
+	)
 	(global_label "USART1_RX"
 		(shape input)
@@
 		)
 	)
+	(global_label "~{SLEEP}"
+		(shape input)
+		(at 138.43 149.86 0)
+		(fields_autoplaced yes)
+		(effects
+			(font
+				(size 1.27 1.27)
+			)
+			(justify left)
+		)
+		(property "Intersheetrefs" "${INTERSHEET_REFS}"
+			(at 147.2208 149.86 0)
+			(effects
+				(font
+					(size 1.27 1.27)
+				)
+				(justify left)
+				(hide yes)
+			)
+		)
+	)
 	(global_label "~{EN}"
 		(shape input)
@@
 		)
 	)
+	(global_label "~{RESET}"
+		(shape input)
+		(at 138.43 147.32 0)
+		(fields_autoplaced yes)
+		(effects
+			(font
+				(size 1.27 1.27)
+			)
+			(justify left)
+		)
+		(property "Intersheetrefs" "${INTERSHEET_REFS}"
+			(at 147.1603 147.32 0)
+			(effects
+				(font
+					(size 1.27 1.27)
+				)
+				(justify left)
+				(hide yes)
+			)
+		)
+	)
 	(global_label "SWCLK"
 		(shape input)
@@
 	(global_label "~{EN}"
 		(shape input)
-		(at 39.37 106.68 0)
+		(at 39.37 105.41 0)
 		(fields_autoplaced yes)
 		(effects
@@
 		)
 		(property "Intersheetrefs" "${INTERSHEET_REFS}"
-			(at 44.8347 106.68 0)
+			(at 44.8347 105.41 0)
 			(effects
 				(font
@@
 		)
 	)
+	(global_label "M2"
+		(shape input)
+		(at 39.37 118.11 0)
+		(fields_autoplaced yes)
+		(effects
+			(font
+				(size 1.27 1.27)
+			)
+			(justify left)
+		)
+		(property "Intersheetrefs" "${INTERSHEET_REFS}"
+			(at 45.0161 118.11 0)
+			(effects
+				(font
+					(size 1.27 1.27)
+				)
+				(justify left)
+				(hide yes)
+			)
+		)
+	)
 	(global_label "USART2_RX"
 		(shape input)
@@
 		)
 	)
+	(global_label "~{SLEEP}"
+		(shape input)
+		(at 39.37 107.95 0)
+		(fields_autoplaced yes)
+		(effects
+			(font
+				(size 1.27 1.27)
+			)
+			(justify left)
+		)
+		(property "Intersheetrefs" "${INTERSHEET_REFS}"
+			(at 48.1608 107.95 0)
+			(effects
+				(font
+					(size 1.27 1.27)
+				)
+				(justify left)
+				(hide yes)
+			)
+		)
+	)
 	(global_label "SPI3_MISO"
 		(shape input)
@@
 		)
 		(pin "~{EN}" input
-			(at 33.02 106.68 0)
+			(at 33.02 105.41 0)
+			(effects
+				(font
+					(size 1.27 1.27)
+				)
+				(justify right)
+			)
+		)
+		(pin "M2" input
+			(at 33.02 118.11 0)
+			(effects
+				(font
+					(size 1.27 1.27)
+				)
+				(justify right)
+			)
+		)
+		(pin "~{RESET}" input
+			(at 33.02 110.49 0)
+			(effects
+				(font
+					(size 1.27 1.27)
+				)
+				(justify right)
+			)
+		)
+		(pin "~{SLEEP}" input
+			(at 33.02 107.95 0)
 			(effects
 				(font

Commit message: Gantry Concept 1 Completion and PCB schematic update
Other:
- moved on the sheet: H1, H2, H3, H4, J11, J13, J7, J9

Commit message: Rough PCB Design Completion
Parts:
- H1, H2, H3, H4: footprint MountingHole:MountingHole_3.2mm_M3_Pad -> MountingHole:MountingHole_4.3mm_M4_Pad
Changed lines of the file:
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@@
 			)
 		)
-		(property "Footprint" "MountingHole:MountingHole_3.2mm_M3_Pad"
+		(property "Footprint" "MountingHole:MountingHole_4.3mm_M4_Pad"
 			(at 121.92 193.04 0)
 			(effects
@@
 			)
 		)
-		(property "Footprint" "MountingHole:MountingHole_3.2mm_M3_Pad"
+		(property "Footprint" "MountingHole:MountingHole_4.3mm_M4_Pad"
 			(at 144.78 193.04 0)
 			(effects
@@
 			)
 		)
-		(property "Footprint" "MountingHole:MountingHole_3.2mm_M3_Pad"
+		(property "Footprint" "MountingHole:MountingHole_4.3mm_M4_Pad"
 			(at 99.06 193.04 0)
 			(effects
@@
 			)
 		)
-		(property "Footprint" "MountingHole:MountingHole_3.2mm_M3_Pad"
+		(property "Footprint" "MountingHole:MountingHole_4.3mm_M4_Pad"
 			(at 76.2 193.04 0)
 			(effects

Commit message: PCB Catastrophe
Connections:
- net GND: now also SW2.1; no longer SW2.2
- net NRST: now also SW2.2; no longer SW2.1
Changed lines of the file:
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@@
+	)
+	(symbol
+		(lib_id "Switch:SW_Push")
+		(at 31.75 52.07 90)
+		(unit 1)
+		(exclude_from_sim no)
+		(in_bom yes)
+		(on_board yes)
+		(dnp no)
+		(fields_autoplaced yes)
+		(property "Reference" "SW2"
+			(at 33.02 50.7999 90)
+			(effects
+				(font
+					(size 1.27 1.27)
+				)
+				(justify right)
+			)
+		)
+		(property "Value" "SW_Push"
+			(at 33.02 53.3399 90)
+			(effects
+				(font
+					(size 1.27 1.27)
+				)
+				(justify right)
+			)
+		)
+		(property "Footprint" "Button_Switch_THT:SW_PUSH_6mm"
+			(at 26.67 52.07 0)
+			(effects
+				(font
+					(size 1.27 1.27)
+				)
+				(hide yes)
+			)
+		)
+		(property "Datasheet" "~"
+			(at 26.67 52.07 0)
+			(effects
+				(font
+					(size 1.27 1.27)
+				)
+				(hide yes)
+			)
+		)
+		(property "Description" "Push button switch, generic, two pins"
+			(at 31.75 52.07 0)
+			(effects
+				(font
+					(size 1.27 1.27)
+				)
+				(hide yes)
+			)
+		)
+		(pin "1"
+		)
+		(pin "2"
+		)
+		(instances
+			(project ""
+				(path "/01596983-65d8-4ce5-b1db-2b179549cf8e"
+					(reference "SW2")
+					(unit 1)
+				)
+			)
+		)
 	)
 	(symbol
@@
 					(unit 1)
 				)
-			)
-		)
-	)
-	(symbol
-		(lib_id "Switch:SW_Push")
-		(at 31.75 52.07 270)
-		(unit 1)
-		(exclude_from_sim no)
-		(in_bom yes)
-		(on_board yes)
-		(dnp no)
-		(fields_autoplaced yes)
-		(property "Reference" "SW2"
-			(at 35.56 50.7999 90)
-			(effects
-				(font
-					(size 1.27 1.27)
-				)
-				(justify left)
-			)
-		)
-		(property "Value" "SW_Push"
-			(at 35.56 53.3399 90)
-			(effects
-				(font
-					(size 1.27 1.27)
-				)
-				(justify left)
-			)
-		)
-		(property "Footprint" "Button_Switch_THT:SW_PUSH_6mm"
-			(at 36.83 52.07 0)
-			(effects
-				(font
-					(size 1.27 1.27)
-				)
-				(hide yes)
-			)
-		)
-		(property "Datasheet" "~"
-			(at 36.83 52.07 0)
-			(effects
-				(font
-					(size 1.27 1.27)
-				)
-				(hide yes)
-			)
-		)
-		(property "Description" "Push button switch, generic, two pins"
-			(at 31.75 52.07 0)
-			(effects
-				(font
-					(size 1.27 1.27)
-				)
-				(hide yes)
-			)
-		)
-		(pin "2"
-		)
-		(pin "1"
-		)
-		(instances
-			(project ""
-				(path "/01596983-65d8-4ce5-b1db-2b179549cf8e"
-					(reference "SW2")
-					(unit 1)
-				)
