File: Hardware/PCB/KiCad_Files/HydrogelBioprinter/Stepper.kicad_sch (KiCad schematic)
At the start: 26 parts, among them J21 Conn_01x04_Pin, J22 Conn_01x04_Pin, J23 Conn_01x04_Pin, J24 Conn_01x04_Pin, J25 Conn_01x04_Pin

Commit message: Schematic Update, PCB preliminary layout, Machine Design addition, and LaTeX report addition
Parts:
- removed A10, A4, A6, A8, A9: MKS TMC2209, Module:Pololu_Breakout-16_15.2x20.3mm, symbol Driver_Motor:Pololu_Breakout_DRV8825
- removed D10, D11, D7, D8, D9: SMAJ28A, Diode_SMD:D_SMA, symbol Diode:SMAJ28A
- added A1, A2, A3, A4, A5: MKS TMC2209, Module:Pololu_Breakout-16_15.2x20.3mm, symbol Driver_Motor:Pololu_Breakout_A4988
- added D10, D6, D7, D8, D9: SMAJ16A, Diode_SMD:D_SMA, symbol Diode:SMAJ16A
- added J22, J24, J26, J28, J30: Conn, Connector_Wire:SolderWire-0.75sqmm_1x02_P4.8mm_D1.25mm_OD2.3mm, symbol Connector_Generic:Conn_01x02
- added J23, J25, J27, J29, J31: Conn, Connector_Wire:SolderWire-0.75sqmm_1x02_P4.8mm_D1.25mm_OD2.3mm, symbol Connector_Generic:Conn_01x01
- added JP1, JP2, JP3, JP4, JP5: Jumper_2_Bridged, TestPoint:TestPoint_Bridge_Pitch2.54mm_Drill0.7mm, symbol Jumper:Jumper_2_Bridged
- C26: renamed from C21; footprint Capacitor_SMD:C_0402_1005Metric -> Capacitor_SMD:C_0603_1608Metric
- C27: renamed from C22; footprint Capacitor_SMD:C_0402_1005Metric -> Capacitor_SMD:C_0603_1608Metric
- C28: renamed from C23; footprint Capacitor_SMD:C_0402_1005Metric -> Capacitor_SMD:C_0603_1608Metric
- C29: renamed from C24; footprint Capacitor_SMD:C_0402_1005Metric -> Capacitor_SMD:C_0603_1608Metric
- C30: renamed from C25; footprint Capacitor_SMD:C_0402_1005Metric -> Capacitor_SMD:C_0603_1608Metric
- J17: renamed from J25; footprint (none) -> Connector_PinHeader_2.54mm:PinHeader_1x04_P2.54mm_Vertical
- J18: renamed from J24; footprint (none) -> Connector_PinHeader_2.54mm:PinHeader_1x04_P2.54mm_Vertical
- J19: renamed from J23; footprint (none) -> Connector_PinHeader_2.54mm:PinHeader_1x04_P2.54mm_Vertical
- J20: renamed from J22; footprint (none) -> Connector_PinHeader_2.54mm:PinHeader_1x04_P2.54mm_Vertical
- J21: footprint (none) -> Connector_PinHeader_2.54mm:PinHeader_1x04_P2.54mm_Vertical
- R17: renamed from R39; value 100K -> 100k; footprint (none) -> Resistor_SMD:R_0805_2012Metric
- renumbered C26 to C31, C27 to C32, C28 to C33, C29 to C34, C30 to C35
Connections:
- net +12V: now also A1.8 (VMOT), A2.8 (VMOT), A3.8 (VMOT), A4.8 (VMOT), A5.8 (VMOT), D10.1 (A1), D6.1 (A1), D7.1 (A1), D8.1 (A1), D9.1 (A1)
- net +3.3V: now also JP1.2 (B), JP2.2 (B), JP3.2 (B), JP4.2 (B), JP5.2 (B); no longer C26.2, C27.2, C28.2, C29.2, C30.2
- net DIR1: now also A1.16 (DIR)
- net DIR2: now also A2.16 (DIR)
- net DIR3: now also A3.16 (DIR)
- net DIR4: now also A4.16 (DIR)
- net DIR5: now also A5.16 (DIR)
- net GND: now also A1.1 (GND), A1.7 (GND), A2.1 (GND), A2.7 (GND), A3.1 (GND), A3.7 (GND), A4.1 (GND), A4.7 (GND), A5.1 (GND), A5.7 (GND), D10.2 (A2), D6.2 (A2), D7.2 (A2), D8.2 (A2), D9.2 (A2)
- net M0: now also A1.10 (MS1), A2.10 (MS1), A3.10 (MS1), A4.10 (MS1), A5.10 (MS1)
- net M1: now also A1.11 (MS2), A2.11 (MS2), A3.11 (MS2), A4.11 (MS2), A5.11 (MS2)
- net STEP1: now also A1.15 (STEP)
- net STEP2: now also A2.15 (STEP)
- net STEP3: now also A3.15 (STEP)
- net STEP4: now also A4.15 (STEP)
- net STEP5: now also A5.15 (STEP)
- net ~{EN}: now also A1.9 (~{ENABLE}), A2.9 (~{ENABLE}), A3.9 (~{ENABLE}), A4.9 (~{ENABLE}), A5.9 (~{ENABLE})
- net at J21.3 (Pin_3): now also A5.4 (1A)
- net at J21.4 (Pin_4): now also A5.3 (1B)
- net at J21.2 (Pin_2): now also A5.5 (2A)
- net at J21.1 (Pin_1): now also A5.6 (2B)
- net at J17.3 (Pin_3): now also A1.4 (1A)
- net at J17.4 (Pin_4): now also A1.3 (1B)
- net at J17.2 (Pin_2): now also A1.5 (2A)
- net at J17.1 (Pin_1): now also A1.6 (2B)
- net at J19.3 (Pin_3): now also A3.4 (1A)
- net at J19.4 (Pin_4): now also A3.3 (1B)
- net at J19.2 (Pin_2): now also A3.5 (2A)
- net at J19.1 (Pin_1): now also A3.6 (2B)
- net at J18.3 (Pin_3): now also A2.4 (1A)
- net at J18.4 (Pin_4): now also A2.3 (1B)
- net at J18.2 (Pin_2): now also A2.5 (2A)
- net at J18.1 (Pin_1): now also A2.6 (2B)
- net at J20.1 (Pin_1): now also A4.6 (2B)
- net at J20.2 (Pin_2): now also A4.5 (2A)
- net at J20.3 (Pin_3): now also A4.4 (1A)
- net at J20.4 (Pin_4): now also A4.3 (1B)
- new net: A5.2 (VDD), C30.2, JP5.1 (A)
- new net: A4.12 (MS3), J29.1 (Pin_1)
- new net: A2.2 (VDD), C27.2, JP2.1 (A)
- new net: A2.12 (MS3), J25.1 (Pin_1)
- new net: A1.2 (VDD), C26.2, JP1.1 (A)
- new net: A5.12 (MS3), J31.1 (Pin_1)
- new net: A5.13 (~{RESET}), J30.2 (Pin_2)
- new net: A5.14 (~{SLEEP}), J30.1 (Pin_1)
- new net: A1.14 (~{SLEEP}), J22.1 (Pin_1)
- new net: A1.13 (~{RESET}), J22.2 (Pin_2)
- new net: A3.12 (MS3), J27.1 (Pin_1)
- new net: A3.13 (~{RESET}), J26.2 (Pin_2)
- new net: A3.14 (~{SLEEP}), J26.1 (Pin_1)
- new net: A3.2 (VDD), C28.2, JP3.1 (A)
- new net: A4.2 (VDD), C29.2, JP4.1 (A)
- new net: A2.14 (~{SLEEP}), J24.1 (Pin_1)
- new net: A2.13 (~{RESET}), J24.2 (Pin_2)
- new net: A4.14 (~{SLEEP}), J28.1 (Pin_1)
- new net: A4.13 (~{RESET}), J28.2 (Pin_2)
- new net: A1.12 (MS3), J23.1 (Pin_1)
- no-connect marks 15 -> 0
Other:
- note added: "Note: In the event that the MKS TMC2209 are unable to be procured, cheap available alternatives such as the A4988 and DRV8825 drivers can be used. If these alternatives are used, then ~{RST} and ~{SLP} pins will need to be pulled high using a spare GPIO or with the 3.3V source and the M2 pin will need to be connected to a spare GPIO pin for microstep setting selection. Solder connection points mu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"
- moved on the sheet: C26, C27, C28, C29, C30, J17, J18, J19, J20, J21

Commit message: Gantry Concept 2 Completion
Parts:
- removed J22, J24, J26, J28, J30: Conn, Connector_Wire:SolderWire-0.75sqmm_1x02_P4.8mm_D1.25mm_OD2.3mm, symbol Connector_Generic:Conn_01x02
- removed J23, J25, J27, J29, J31: Conn, Connector_Wire:SolderWire-0.75sqmm_1x02_P4.8mm_D1.25mm_OD2.3mm, symbol Connector_Generic:Conn_01x01
Connections:
- net M2: now reaches A4.12 (MS3)
- net M2: now also A1.12 (MS3), A2.12 (MS3), A3.12 (MS3), A5.12 (MS3)
- net ~{RESET}: now reaches A5.13 (~{RESET})
- net ~{RESET}: now also A1.13 (~{RESET}), A2.13 (~{RESET}), A3.13 (~{RESET}), A4.13 (~{RESET})
- net ~{SLEEP}: now reaches A5.14 (~{SLEEP})
- net ~{SLEEP}: now also A1.14 (~{SLEEP}), A2.14 (~{SLEEP}), A3.14 (~{SLEEP}), A4.14 (~{SLEEP})

Commit message: Gantry Concept 1 Completion and PCB schematic update
Changed lines of the file:
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@@
 	(wire
 		(pts
-			(xy 33.02 112.395) (xy 33.02 114.3)
+			(xy 33.02 113.03) (xy 33.02 114.3)
 		)
 		(stroke
@@
 	(wire
 		(pts
-			(xy 48.26 101.6) (xy 48.26 103.505)
+			(xy 48.26 101.6) (xy 48.26 104.14)
 		)
 		(stroke
@@
 	(wire
 		(pts
-			(xy 45.72 99.06) (xy 45.72 103.505)
+			(xy 45.72 99.06) (xy 45.72 104.14)
 		)
 		(stroke
@@
 	(hierarchical_label "~{SLEEP}"
 		(shape input)
-		(at 48.26 103.505 270)
+		(at 48.26 104.14 270)
 		(effects
 			(font
@@
 	(hierarchical_label "~{RESET}"
 		(shape input)
-		(at 45.72 103.505 270)
+		(at 45.72 104.14 270)
 		(effects
 			(font
@@
 	(symbol
 		(lib_id "power:+3.3V")
-		(at 33.02 112.395 0)
+		(at 33.02 113.03 0)
 		(mirror y)
 		(unit 1)
@@
 		(fields_autoplaced yes)
 		(property "Reference" "#PWR069"
-			(at 33.02 116.205 0)
+			(at 33.02 116.84 0)
 			(effects
 				(font
@@
 		)
 		(property "Value" "+3.3V"
-			(at 33.02 107.315 0)
+			(at 33.02 107.95 0)
 			(effects
 				(font
@@
 		)
 		(property "Footprint" ""
-			(at 33.02 112.395 0)
+			(at 33.02 113.03 0)
 			(effects
 				(font
@@
 		)
 		(property "Datasheet" ""
-			(at 33.02 112.395 0)
+			(at 33.02 113.03 0)
 			(effects
 				(font
@@
 		)
 		(property "Description" "Power symbol creates a global label with name \"+3.3V\""
-			(at 33.02 112.395 0)
-			(effects
-				(font
+			(at 33.02 113.03 0)
+			(effects
+				(font

Commit message: Final PCB Design
Parts:
- JP1, JP2, JP3, JP4, JP5: footprint TestPoint:TestPoint_Bridge_Pitch2.54mm_Drill0.7mm -> TestPoint:TestPoint_2Pads_Pitch2.54mm_Drill0.8mm
Changed lines of the file:
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@@
 	(wire
 		(pts
-			(xy 223.52 90.17) (xy 223.52 91.44)
-		)
-		(stroke
-			(width 0)
-			(type default)
-		)
-	)
-	(wire
-		(pts
 			(xy 68.58 74.93) (xy 68.58 125.73)
 		)
@@
 	(wire
 		(pts
+			(xy 223.52 90.17) (xy 223.52 91.44)
+		)
+		(stroke
+			(width 0)
+			(type default)
+		)
+	)
+	(wire
+		(pts
 			(xy 195.58 74.93) (xy 195.58 90.17)
 		)
@@
 			)
 		)
-		(property "Footprint" "TestPoint:TestPoint_Bridge_Pitch2.54mm_Drill0.7mm"
+		(property "Footprint" "TestPoint:TestPoint_2Pads_Pitch2.54mm_Drill0.8mm"
 			(at 86.36 85.09 0)
 			(effects
@@
 			)
 		)
-		(property "Footprint" "TestPoint:TestPoint_Bridge_Pitch2.54mm_Drill0.7mm"
+		(property "Footprint" "TestPoint:TestPoint_2Pads_Pitch2.54mm_Drill0.8mm"
 			(at 223.52 85.09 0)
 			(effects
@@
 			)
 		)
-		(property "Footprint" "TestPoint:TestPoint_Bridge_Pitch2.54mm_Drill0.7mm"
+		(property "Footprint" "TestPoint:TestPoint_2Pads_Pitch2.54mm_Drill0.8mm"
 			(at 38.1 85.09 0)
 			(effects
@@
 			)
 		)
-		(property "Footprint" "TestPoint:TestPoint_Bridge_Pitch2.54mm_Drill0.7mm"
+		(property "Footprint" "TestPoint:TestPoint_2Pads_Pitch2.54mm_Drill0.8mm"
 			(at 132.08 85.09 0)
 			(effects
@@
 	)
 	(symbol
+		(lib_id "power:+3.3V")
+		(at 223.52 91.44 180)
+		(unit 1)
+		(exclude_from_sim no)
+		(in_bom yes)
+		(on_board yes)
+		(dnp no)
+		(fields_autoplaced yes)
+		(property "Reference" "#PWR020"
+			(at 223.52 87.63 0)
+			(effects
+				(font
+					(size 1.27 1.27)
+				)
+				(hide yes)
+			)
+		)
+		(property "Value" "+3.3V"
+			(at 223.52 96.52 0)
+			(effects
+				(font
+					(size 1.27 1.27)
+				)
+			)
+		)
+		(property "Footprint" ""
+			(at 223.52 91.44 0)
+			(effects
+				(font
+					(size 1.27 1.27)
+				)
+				(hide yes)
+			)
+		)
+		(property "Datasheet" ""
+			(at 223.52 91.44 0)
+			(effects
+				(font
+					(size 1.27 1.27)
+				)
+				(hide yes)
+			)
+		)
+		(property "Description" "Power symbol creates a global label with name \"+3.3V\""
+			(at 223.52 91.44 0)
+			(effects
+				(font
+					(size 1.27 1.27)
+				)
+				(hide yes)
+			)
+		)
+		(pin "1"
+		)
+		(instances
+			(project ""
+				(path "/01596983-65d8-4ce5-b1db-2b179549cf8e/e55b0dd9-1440-4979-bba0-bc15e307ee78"
+					(reference "#PWR020")
+					(unit 1)
+				)
+			)
+		)
+	)
+	(symbol
 		(lib_id "power:GND")
 		(at 149.86 157.48 0)
@@
 	)
 	(symbol
-		(lib_id "power:+3.3V")
-		(at 223.52 91.44 180)
-		(unit 1)
-		(exclude_from_sim no)
-		(in_bom yes)
-		(on_board yes)
-		(dnp no)
-		(fields_autoplaced yes)
-		(property "Reference" "#PWR068"
-			(at 223.52 87.63 0)
-			(effects
-				(font
-					(size 1.27 1.27)
-				)
-				(hide yes)
-			)
-		)
-		(property "Value" "+3.3V"
-			(at 223.52 96.52 0)
-			(effects
-				(font
-					(size 1.27 1.27)
-				)
-			)
-		)
-		(property "Footprint" ""
-			(at 223.52 91.44 0)
-			(effects
-				(font
-					(size 1.27 1.27)
-				)
-				(hide yes)
-			)
-		)
-		(property "Datasheet" ""
-			(at 223.52 91.44 0)
-			(effects
-				(font
-					(size 1.27 1.27)
-				)
-				(hide yes)
-			)
-		)
-		(property "Description" "Power symbol creates a global label with name \"+3.3V\""
-			(at 223.52 91.44 0)
-			(effects
-				(font
-					(size 1.27 1.27)
-				)
-				(hide yes)
-			)
-		)
-		(pin "1"
-		)
-		(instances
-			(project "HydrogelBioprinter"
-				(path "/01596983-65d8-4ce5-b1db-2b179549cf8e/e55b0dd9-1440-4979-bba0-bc15e307ee78"
-					(reference "#PWR068")
-					(unit 1)
-				)
-			)
-		)
-	)
-	(symbol
 		(lib_id "power:+24V")
 		(at 241.3 147.32 0)
@@
 			)
 		)
-		(property "Footprint" "TestPoint:TestPoint_Bridge_Pitch2.54mm_Drill0.7mm"
+		(property "Footprint" "TestPoint:TestPoint_2Pads_Pitch2.54mm_Drill0.8mm"
 			(at 177.8 85.09 0)
 			(effects

Commit message: PCB Catastrophe
Parts:
- A1, A2, A3, A4, A5: value MKS TMC2209 -> A4988
Changed lines of the file:
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@@
 			)
 		)
-		(property "Value" "MKS TMC2209"
-			(at 255.27 53.086 90)
+		(property "Value" "A4988"
+			(at 251.46 53.34 90)
 			(effects
 				(font
@@
 			)
 		)
-		(property "Value" "MKS TMC2209"
-			(at 163.83 53.086 90)
+		(property "Value" "A4988"
+			(at 160.02 53.34 90)
 			(effects
 				(font
@@
 			)
 		)
-		(property "Value" "MKS TMC2209"
-			(at 69.85 53.086 90)
+		(property "Value" "A4988"
+			(at 66.04 53.34 90)
 			(effects
 				(font
@@
 			)
 		)
-		(property "Value" "MKS TMC2209"
-			(at 209.55 53.086 90)
+		(property "Value" "A4988"
+			(at 205.74 53.34 90)
 			(effects
 				(font
@@
 			)
 		)
-		(property "Value" "MKS TMC2209"
-			(at 118.11 53.086 90)
-			(effects
-				(font
+		(property "Value" "A4988"
+			(at 114.3 53.34 90)
+			(effects
+				(font
